File: boards/kossel_mini_extruder.sch (EAGLE design)
At the start: 34 parts

Commit message: made vias beefier for hand soldering
Parts:
- removed LOGO1: OSHW-LOGOS, SparkFun-Aesthetics:OSHW-LOGOS
Changed lines of the file:
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@@
 <part name="GND1" library="SparkFun-Aesthetics" deviceset="GND" device=""/>
 <part name="GND3" library="SparkFun-Aesthetics" deviceset="GND" device=""/>
-<part name="LOGO1" library="SparkFun-Aesthetics" deviceset="OSHW-LOGO" device="S"/>
 <part name="LED7" library="SparkFun-LED" deviceset="LED" device="0805"/>
 <part name="LED8" library="SparkFun-LED" deviceset="LED" device="0805"/>
@@
 <instance part="GND1" gate="1" x="22.86" y="50.8"/>
 <instance part="GND3" gate="1" x="-17.78" y="43.18"/>
-<instance part="LOGO1" gate="G$1" x="-20.32" y="91.44"/>
 <instance part="LED7" gate="G$1" x="-22.86" y="33.02"/>
 <instance part="LED8" gate="G$1" x="-12.7" y="33.02"/>

Commit message: replaced 2x5 header with 2x4 header
Parts:
- removed HOT_HEADER: M05X2RA, SparkFun-Connectors:M05X2RA
- added SV1: (no value), con-lstb:MA04-2
Connections:
- net FAN_VCC: now also SV1.6; no longer HOT_HEADER.3
- net GND: now also SV1.4; no longer HOT_HEADER.5, HOT_HEADER.6
- net N$10: now also SV1.1; no longer HOT_HEADER.10, HOT_HEADER.8
- net N$11: now also SV1.3; no longer HOT_HEADER.9
- net N$12: now also SV1.2; no longer HOT_HEADER.7
- net N$15: now also SV1.7; no longer HOT_HEADER.2, HOT_HEADER.4
- net N$17: now also SV1.8; no longer HOT_HEADER.1
Changed lines of the file:
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@@
 <part name="GND5" library="SparkFun-Aesthetics" deviceset="GND" device=""/>
 <part name="HOT_12V" library="OBKP_Effector_PCB" deviceset="LUG" device="3-X"/>
-<part name="HOT_HEADER" library="SparkFun-Connectors" deviceset="M05X2" device="RA"/>
 <part name="PROBE_GND" library="OBKP_Effector_PCB" deviceset="LUG" device="3-X"/>
 <part name="PROBE_SIG" library="OBKP_Effector_PCB" deviceset="LUG" device="3-X"/>
+<part name="SV1" library="con-lstb" deviceset="MA04-2" device=""/>
 </parts>
 <sheets>
@@
 <attribute name="NAME" x="76.2" y="68.58" size="1.778" layer="95"/>
 </instance>
-<instance part="HOT_HEADER" gate="G$1" x="38.1" y="73.66"/>
 <instance part="PROBE_GND" gate="G$1" x="63.5" y="93.98" smashed="yes" rot="R270">
 <attribute name="NAME" x="76.2" y="93.98" size="1.778" layer="95"/>
@@
 <attribute name="NAME" x="76.2" y="101.6" size="1.778" layer="95"/>
 </instance>
+<instance part="SV1" gate="G$1" x="38.1" y="76.2"/>
 </instances>
 <busses>
@@
 <pinref part="GND1" gate="1" pin="GND"/>
 <wire x1="22.86" y1="53.34" x2="22.86" y2="55.88" width="0.1524" layer="91"/>
-<pinref part="HOT_HEADER" gate="G$1" pin="5"/>
 <wire x1="22.86" y1="55.88" x2="22.86" y2="73.66" width="0.1524" layer="91"/>
 <wire x1="22.86" y1="73.66" x2="30.48" y2="73.66" width="0.1524" layer="91"/>
-<pinref part="HOT_HEADER" gate="G$1" pin="6"/>
-<wire x1="45.72" y1="73.66" x2="48.26" y2="73.66" width="0.1524" layer="91"/>
-<wire x1="48.26" y1="73.66" x2="48.26" y2="55.88" width="0.1524" layer="91"/>
 <wire x1="48.26" y1="55.88" x2="22.86" y2="55.88" width="0.1524" layer="91"/>
 <junction x="22.86" y="55.88"/>
@@
 <wire x1="60.96" y1="93.98" x2="60.96" y2="55.88" width="0.1524" layer="91"/>
 <wire x1="60.96" y1="55.88" x2="48.26" y2="55.88" width="0.1524" layer="91"/>
+<pinref part="SV1" gate="G$1" pin="4"/>
 </segment>
 </net>
@@
 <junction x="7.62" y="76.2"/>
 <wire x1="15.24" y1="38.1" x2="15.24" y2="76.2" width="0.1524" layer="91"/>
-<pinref part="HOT_HEADER" gate="G$1" pin="3"/>
 <wire x1="15.24" y1="76.2" x2="30.48" y2="76.2" width="0.1524" layer="91"/>
 <junction x="15.24" y="76.2"/>
+<pinref part="SV1" gate="G$1" pin="6"/>
 </segment>
 </net>
 <net name="N$10" class="0">
 <segment>
-<pinref part="HOT_HEADER" gate="G$1" pin="10"/>
 <pinref part="HOT_12V" gate="G$1" pin="P$1"/>
-<wire x1="45.72" y1="68.58" x2="53.34" y2="68.58" width="0.1524" layer="91"/>
 <wire x1="53.34" y1="68.58" x2="63.5" y2="68.58" width="0.1524" layer="91"/>
-<wire x1="53.34" y1="68.58" x2="53.34" y2="71.12" width="0.1524" layer="91"/>
-<pinref part="HOT_HEADER" gate="G$1" pin="8"/>
-<wire x1="53.34" y1="71.12" x2="45.72" y2="71.12" width="0.1524" layer="91"/>
-<junction x="53.34" y="68.58"/>
-<junction x="53.34" y="71.12"/>
 <pinref part="FAN_0_12V" gate="G$1" pin="P$1"/>
 <wire x1="53.34" y1="93.98" x2="53.34" y2="96.52" width="0.1524" layer="91"/>
@@
 <wire x1="38.1" y1="93.98" x2="45.72" y2="93.98" width="0.1524" layer="91"/>
 <junction x="53.34" y="93.98"/>
+<wire x1="53.34" y1="68.58" x2="53.34" y2="71.12" width="0.1524" layer="91"/>
+<junction x="53.34" y="71.12"/>
 <wire x1="53.34" y1="71.12" x2="53.34" y2="93.98" width="0.1524" layer="91"/>
+<pinref part="SV1" gate="G$1" pin="1"/>
+<wire x1="45.72" y1="71.12" x2="53.34" y2="71.12" width="0.1524" layer="91"/>
 </segment>
 </net>
@@
 <segment>
 <pinref part="THERM_SIG" gate="G$1" pin="P$1"/>
-<wire x1="63.5" y1="58.42" x2="27.94" y2="58.42" width="0.1524" layer="91"/>
-<wire x1="27.94" y1="58.42" x2="27.94" y2="68.58" width="0.1524" layer="91"/>
-<pinref part="HOT_HEADER" gate="G$1" pin="9"/>
-<wire x1="27.94" y1="68.58" x2="30.48" y2="68.58" width="0.1524" layer="91"/>
+<wire x1="63.5" y1="58.42" x2="50.8" y2="58.42" width="0.1524" layer="91"/>
+<pinref part="SV1" gate="G$1" pin="3"/>
+<wire x1="45.72" y1="73.66" x2="50.8" y2="73.66" width="0.1524" layer="91"/>
+<wire x1="50.8" y1="73.66" x2="50.8" y2="58.42" width="0.1524" layer="91"/>
 </segment>
 </net>
@@
 <wire x1="58.42" y1="83.82" x2="25.4" y2="83.82" width="0.1524" layer="91"/>
 <wire x1="25.4" y1="83.82" x2="25.4" y2="71.12" width="0.1524" layer="91"/>
-<pinref part="HOT_HEADER" gate="G$1" pin="7"/>
 <wire x1="25.4" y1="71.12" x2="30.48" y2="71.12" width="0.1524" layer="91"/>
+<pinref part="SV1" gate="G$1" pin="2"/>
 </segment>
 </net>
@@
 <junction x="20.32" y="93.98"/>
 <junction x="27.94" y="93.98"/>
-<pinref part="HOT_HEADER" gate="G$1" pin="1"/>
 <wire x1="30.48" y1="78.74" x2="27.94" y2="78.74" width="0.1524" layer="91"/>
 <wire x1="27.94" y1="78.74" x2="27.94" y2="93.98" width="0.1524" layer="91"/>
+<pinref part="SV1" gate="G$1" pin="8"/>
 </segment>
 </net>
 <net name="N$15" class="0">
 <segment>
-<pinref part="HOT_HEADER" gate="G$1" pin="2"/>
-<wire x1="45.72" y1="78.74" x2="50.8" y2="78.74" width="0.1524" layer="91"/>
 <pinref part="HOT_PWM" gate="G$1" pin="P$1"/>
-<wire x1="50.8" y1="78.74" x2="63.5" y2="78.74" width="0.1524" layer="91"/>
-<wire x1="50.8" y1="78.74" x2="50.8" y2="76.2" width="0.1524" layer="91"/>
-<pinref part="HOT_HEADER" gate="G$1" pin="4"/>
-<wire x1="50.8" y1="76.2" x2="45.72" y2="76.2" width="0.1524" layer="91"/>
-<junction x="50.8" y="78.74"/>
-</segment>
-</net>
+<wire x1="45.72" y1="78.74" x2="63.5" y2="78.74" width="0.1524" layer="91"/>
+<pinref part="SV1" gate="G$1" pin="7"/>
+</segment>
+</net>

Commit message: put fan on separate 12V supply line
Connections:
- removed net N$10: FAN_0_12V.P$1, FAN_1_12V.P$1, FAN_2_12V.P$1, HOT_12V.P$1, SV1.1
- new net FAN_12V: FAN_0_12V.P$1, FAN_1_12V.P$1, FAN_2_12V.P$1, SV1.5
- new net HOT_12V: HOT_12V.P$1, SV1.1
Changed lines of the file:
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@@
 </segment>
 </net>
-<net name="N$10" class="0">
+<net name="FAN_12V" class="0">
 <segment>
-<pinref part="HOT_12V" gate="G$1" pin="P$1"/>
-<wire x1="53.34" y1="68.58" x2="63.5" y2="68.58" width="0.1524" layer="91"/>
 <pinref part="FAN_0_12V" gate="G$1" pin="P$1"/>
 <wire x1="53.34" y1="93.98" x2="53.34" y2="96.52" width="0.1524" layer="91"/>
@@
 <wire x1="38.1" y1="93.98" x2="45.72" y2="93.98" width="0.1524" layer="91"/>
 <junction x="53.34" y="93.98"/>
-<wire x1="53.34" y1="68.58" x2="53.34" y2="71.12" width="0.1524" layer="91"/>
-<junction x="53.34" y="71.12"/>
-<wire x1="53.34" y1="71.12" x2="53.34" y2="93.98" width="0.1524" layer="91"/>
-<pinref part="SV1" gate="G$1" pin="1"/>
-<wire x1="45.72" y1="71.12" x2="53.34" y2="71.12" width="0.1524" layer="91"/>
+<wire x1="53.34" y1="93.98" x2="53.34" y2="76.2" width="0.1524" layer="91"/>
+<pinref part="SV1" gate="G$1" pin="5"/>
+<wire x1="53.34" y1="76.2" x2="45.72" y2="76.2" width="0.1524" layer="91"/>
 </segment>
 </net>
@@
 </segment>
 </net>
+<net name="HOT_12V" class="0">
+<segment>
+<pinref part="HOT_12V" gate="G$1" pin="P$1"/>
+<wire x1="53.34" y1="68.58" x2="63.5" y2="68.58" width="0.1524" layer="91"/>
+<wire x1="53.34" y1="68.58" x2="53.34" y2="71.12" width="0.1524" layer="91"/>
+<pinref part="SV1" gate="G$1" pin="1"/>
+<wire x1="45.72" y1="71.12" x2="53.34" y2="71.12" width="0.1524" layer="91"/>
+</segment>
+</net>

Commit message: put fan and hot back on same 12v to make space to breakout thermister gnd
Connections:
- net FAN_VCC renamed VCC
- removed net FAN_12V: FAN_0_12V.P$1, FAN_1_12V.P$1, FAN_2_12V.P$1, SV1.5
- removed net HOT_12V: HOT_12V.P$1, SV1.1
- new net 12V: FAN_0_12V.P$1, FAN_1_12V.P$1, FAN_2_12V.P$1, HOT_12V.P$1, SV1.1
- new net N$8: SV1.5, THERM_GND.P$1
- net GND: no longer THERM_GND.P$1
Changed lines of the file:
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@@
 <wire x1="22.86" y1="55.88" x2="22.86" y2="73.66" width="0.1524" layer="91"/>
 <wire x1="22.86" y1="73.66" x2="30.48" y2="73.66" width="0.1524" layer="91"/>
-<wire x1="48.26" y1="55.88" x2="22.86" y2="55.88" width="0.1524" layer="91"/>
+<wire x1="60.96" y1="55.88" x2="22.86" y2="55.88" width="0.1524" layer="91"/>
 <junction x="22.86" y="55.88"/>
-<pinref part="THERM_GND" gate="G$1" pin="P$1"/>
-<wire x1="63.5" y1="50.8" x2="48.26" y2="50.8" width="0.1524" layer="91"/>
-<wire x1="48.26" y1="50.8" x2="48.26" y2="55.88" width="0.1524" layer="91"/>
-<junction x="48.26" y="55.88"/>
 <pinref part="PROBE_GND" gate="G$1" pin="P$1"/>
 <wire x1="63.5" y1="93.98" x2="60.96" y2="93.98" width="0.1524" layer="91"/>
 <wire x1="60.96" y1="93.98" x2="60.96" y2="55.88" width="0.1524" layer="91"/>
-<wire x1="60.96" y1="55.88" x2="48.26" y2="55.88" width="0.1524" layer="91"/>
 <pinref part="SV1" gate="G$1" pin="4"/>
 </segment>
@@
 </segment>
 </net>
-<net name="FAN_VCC" class="0">
+<net name="VCC" class="0">
 <segment>
 <pinref part="LED10" gate="G$1" pin="A"/>
@@
 </segment>
 </net>
-<net name="FAN_12V" class="0">
-<segment>
-<pinref part="FAN_0_12V" gate="G$1" pin="P$1"/>
-<wire x1="53.34" y1="93.98" x2="53.34" y2="96.52" width="0.1524" layer="91"/>
-<pinref part="FAN_2_12V" gate="G$1" pin="P$1"/>
-<wire x1="45.72" y1="93.98" x2="45.72" y2="96.52" width="0.1524" layer="91"/>
-<wire x1="45.72" y1="93.98" x2="53.34" y2="93.98" width="0.1524" layer="91"/>
-<junction x="45.72" y="93.98"/>
-<pinref part="FAN_1_12V" gate="G$1" pin="P$1"/>
-<wire x1="38.1" y1="96.52" x2="38.1" y2="93.98" width="0.1524" layer="91"/>
-<wire x1="38.1" y1="93.98" x2="45.72" y2="93.98" width="0.1524" layer="91"/>
-<junction x="53.34" y="93.98"/>
-<wire x1="53.34" y1="93.98" x2="53.34" y2="76.2" width="0.1524" layer="91"/>
-<pinref part="SV1" gate="G$1" pin="5"/>
-<wire x1="53.34" y1="76.2" x2="45.72" y2="76.2" width="0.1524" layer="91"/>
-</segment>
-</net>
 <net name="N$11" class="0">
 <segment>
@@
 </segment>
 </net>
-<net name="HOT_12V" class="0">
+<net name="12V" class="0">
 <segment>
+<pinref part="FAN_0_12V" gate="G$1" pin="P$1"/>
+<wire x1="53.34" y1="93.98" x2="53.34" y2="96.52" width="0.1524" layer="91"/>
+<pinref part="FAN_2_12V" gate="G$1" pin="P$1"/>
+<wire x1="45.72" y1="93.98" x2="45.72" y2="96.52" width="0.1524" layer="91"/>
+<wire x1="45.72" y1="93.98" x2="53.34" y2="93.98" width="0.1524" layer="91"/>
+<junction x="45.72" y="93.98"/>
+<pinref part="FAN_1_12V" gate="G$1" pin="P$1"/>
+<wire x1="38.1" y1="96.52" x2="38.1" y2="93.98" width="0.1524" layer="91"/>
+<wire x1="38.1" y1="93.98" x2="45.72" y2="93.98" width="0.1524" layer="91"/>
 <pinref part="HOT_12V" gate="G$1" pin="P$1"/>
 <wire x1="53.34" y1="68.58" x2="63.5" y2="68.58" width="0.1524" layer="91"/>
@@
 <pinref part="SV1" gate="G$1" pin="1"/>
 <wire x1="45.72" y1="71.12" x2="53.34" y2="71.12" width="0.1524" layer="91"/>
+<wire x1="53.34" y1="93.98" x2="53.34" y2="71.12" width="0.1524" layer="91"/>
+<junction x="53.34" y="71.12"/>
+<junction x="53.34" y="93.98"/>
 </segment>
 </net>
+<net name="N$8" class="0">
+<segment>
+<pinref part="THERM_GND" gate="G$1" pin="P$1"/>
+<wire x1="63.5" y1="50.8" x2="48.26" y2="50.8" width="0.1524" layer="91"/>
+<wire x1="48.26" y1="50.8" x2="48.26" y2="76.2" width="0.1524" layer="91"/>
+<pinref part="SV1" gate="G$1" pin="5"/>
+<wire x1="48.26" y1="76.2" x2="45.72" y2="76.2" width="0.1524" layer="91"/>
+</segment>
+</net>

Commit message: removed fan stuff and added red leds
Parts:
- removed FAN_0_12V, FAN_0_PWM, FAN_1_12V, FAN_1_PWM, FAN_2_12V, FAN_2_PWM: LUG2.3, OBKP_Effector_PCB:LUG2.3
- removed LED7: (no value), SparkFun-LED:LED0805
- removed R7: (no value), SparkFun-Passives:RESISTOR0805-RES
- added LED11, LED12, LED13: (no value), SparkFun-LED:LED0805
- added R11, R12, R13: (no value), SparkFun-Passives:RESISTOR0805-RES
Connections:
- removed net 12V: FAN_0_12V.P$1, FAN_1_12V.P$1, FAN_2_12V.P$1, HOT_12V.P$1, SV1.1
- removed net N$7: LED7.C, R7.2
- new net N$10: HOT_12V.P$1, SV1.1
- new net N$16: LED11.C, R11.2
- new net N$18: LED13.C, R13.2
- new net VCC1: LED11.A, LED12.A, LED13.A, SV1.8
- net GND: now also R11.1, R12.1, R13.1; no longer PROBE_GND.P$1, R7.1
- net N$17: now also LED12.C, R12.2; no longer FAN_0_PWM.P$1, FAN_1_PWM.P$1, FAN_2_PWM.P$1, SV1.8
- net N$8: now also PROBE_GND.P$1
- net VCC: no longer LED7.A
